Commit message: edited some gazebo visualization properties

File: kinova_description/urdf/kinova_common.xacro (robot description, xacro)
@@ -43,4 +43,44 @@
 						<xacro:kinova_inertial mesh_no="${mesh_no}"/>
       </link>
+      <gazebo reference="${link_name}">
+        <visual>
+            <material>
+                <ambient>0.19225 0.19225 0.19225 1.0</ambient>
+                <diffuse>0.50754 0.50754 0.50754 1.0</diffuse>
+                <specular>0.508273 0.508273 0.508273 1.0</specular>
+                <emissive>0.0 0.0 0.0 0.0</emissive>
+            </material>
+        </visual>
+      </gazebo>
+      <gazebo reference="j2s7s300_link_finger_1">
+        <visual>
+            <material>
+                <ambient>0.792156862745098 0.819607843137255 0.933333333333333 1.0</ambient>
+                <diffuse>0.792156862745098 0.819607843137255 0.933333333333333 1.0</diffuse>
+                <specular>0.792156862745098 0.819607843137255 0.933333333333333 1.0</specular>
+                <emissive>0.0 0.0 0.0 0.0</emissive>
+            </material>
+        </visual>
+      </gazebo>
+      <gazebo reference="j2s7s300_link_finger_2">
+        <visual>
+            <material>
+                <ambient>0.792156862745098 0.819607843137255 0.933333333333333 1.0</ambient>
+                <diffuse>0.792156862745098 0.819607843137255 0.933333333333333 1.0</diffuse>
+                <specular>0.792156862745098 0.819607843137255 0.933333333333333 1.0</specular>
+                <emissive>0.0 0.0 0.0 0.0</emissive>
+            </material>
+        </visual>
+      </gazebo>
+      <gazebo reference="j2s7s300_link_finger_3">
+        <visual>
+            <material>
+                <ambient>0.792156862745098 0.819607843137255 0.933333333333333 1.0</ambient>
+                <diffuse>0.792156862745098 0.819607843137255 0.933333333333333 1.0</diffuse>
+                <specular>0.792156862745098 0.819607843137255 0.933333333333333 1.0</specular>
+                <emissive>0.0 0.0 0.0 0.0</emissive>
+            </material>
+        </visual>
+      </gazebo>
     </xacro:macro>
   <xacro:macro name="kinova_armjoint" params="joint_name type parent child joint_axis_xyz joint_origin_xyz joint_origin_rpy joint_lower_limit joint_upper_limit fixed:=false">
