Commit message: making gazebo work with kinetic

File: kinova_description/urdf/j2s7s300_standalone.xacro (robot description, xacro)
@@ -19,5 +19,5 @@
       <origin xyz="0 0 0" rpy="0 0 0" />
       <geometry>
-        <box size = "0 0 0"/>
+        <box size = "0.1 0.1 0.1"/>
       </geometry>
     <!--<material name="Black" /> -->
@@ -26,5 +26,5 @@
       <origin xyz="0 0 0" rpy="0 0 0" />
       <geometry>
-        <box size = "0 0 0"/>
+        <box size = "0.1 0.1 0.1"/>
       </geometry>
     </collision>

Commit message: kinova-gazebo fix to make it run on kinetic and gazebo 8!

File: kinova_description/urdf/j2s7s300_standalone.xacro (robot description, xacro)
@@ -19,5 +19,5 @@
       <origin xyz="0 0 0" rpy="0 0 0" />
       <geometry>
-        <box size = "0.1 0.1 0.1"/>
+        <box size = "0.00001 0.00001 0.00001"/>
       </geometry>
     <!--<material name="Black" /> -->
@@ -26,5 +26,5 @@
       <origin xyz="0 0 0" rpy="0 0 0" />
       <geometry>
-        <box size = "0.1 0.1 0.1"/>
+        <box size = "0.00001 0.00001 0.00001"/>
       </geometry>
     </collision>

File: kinova_description/urdf/kinova_common.xacro (robot description, xacro)
@@ -70,10 +70,10 @@
             <visual>
                 <geometry>
-                    <box size = "0 0 0"/>
+                    <box size = "0.00001 0.00001 0.00001"/>
                 </geometry>
             </visual>
             <collision>
                 <geometry>
-                    <box size = "0 0 0"/>
+                    <box size = "0.00001 0.00001 0.00001"/>
                 </geometry>
             </collision>

Commit message: new world, simplified sandbox for easy manipulation

File: kinova_description/urdf/j2s7s300_standalone.xacro (robot description, xacro)
@@ -32,5 +32,5 @@
   <!-- for gazebo -->
   <link name="world"/>
-  <joint name="connect_root_and_world" type="fixed">
+  <joint name="connect_root_and_table" type="fixed">
     <child link="root" />
     <parent link="world" />
